Commit message: feat: for rover

File: sample_vehicle_description/urdf/vehicle.xacro (robot description, xacro)
@@ -1,4 +1,4 @@
 <?xml version="1.0"?>
-<robot xmlns:xacro="http://ros.org/wiki/xacro">
+<robot name="canedudev_rover" xmlns:xacro="http://ros.org/wiki/xacro">
   <!-- load parameter -->
   <xacro:property name="vehicle_info" value="${xacro.load_yaml('$(find sample_vehicle_description)/config/vehicle_info.param.yaml')}"/>
@@ -6,7 +6,7 @@
   <link name="base_link">
     <visual>
-      <origin xyz="${vehicle_info['/**']['ros__parameters']['wheel_base']/2.0} 0 0" rpy="${pi/2.0} 0 ${pi}"/>
+      <origin xyz="${vehicle_info['/**']['ros__parameters']['wheel_base']/2.0} 0 0" rpy="0 0 0"/>
       <geometry>
-        <mesh filename="package://sample_vehicle_description/mesh/lexus.dae" scale="1 1 1"/>
+        <mesh filename="package://sample_vehicle_description/mesh/canedudev_rover.dae" scale="1 1 1"/>
       </geometry>
     </visual>
